Commit message: updated d415 to match intel's new camera_link location

File: realsense_description/urdf/_d415.gazebo.xacro (robot description, xacro)
@@ -3,7 +3,4 @@
 <xacro:macro name="d415_realsense_gazebo"
   params="prefix color_width color_height color_update_rate depth_update_rate">
-  <gazebo reference="${prefix}camera_link">
-    <material value="Gazebo/Grey" />
-  </gazebo>
   <gazebo reference="${prefix}camera_color_frame">
     <sensor type="depth" name="${prefix}">

File: realsense_description/urdf/_d415.urdf.xacro (robot description, xacro)
@@ -31,7 +31,7 @@
       <xacro:insert_block name="origin" />
       <parent link="${parent}"/>
-      <child link="${prefix}camera_link" />
+      <child link="${prefix}camera_bottom_screw_link" />
     </joint>
-    <link name="${prefix}camera_link">
+    <link name="${prefix}camera_bottom_screw_link">
       <visual>
         <origin xyz="0.0 0.0 0.0" rpy="0 0 0"/>
@@ -39,5 +39,4 @@
           <mesh filename="package://realsense_description/meshes/visual/d415.dae" />
         </geometry>
-        <material name="grey"/>
       </visual>
       <collision>
@@ -54,8 +53,14 @@
       </inertial>
     </link>
+    <link name="${prefix}camera_link"/>
+    <joint name="${prefix}camera_link_joint" type="fixed">
+      <origin xyz="${d415_cam_depth_px} ${d415_cam_depth_py} ${d415_cam_depth_pz}" rpy="0 0 0"/>
+      <parent link="${prefix}camera_bottom_screw_link"/>
+      <child link="${prefix}camera_link" />
+    </joint>
     <!-- camera depth joints and links -->
     <joint name="${prefix}camera_depth_joint" type="fixed">
       <origin xyz="${d415_cam_depth_px} ${d415_cam_depth_py} ${d415_cam_depth_pz}" rpy="0 0 0"/>
-      <parent link="${prefix}camera_link"/>
+      <parent link="${prefix}camera_bottom_screw_link"/>
       <child link="${prefix}camera_depth_frame" />
     </joint>

File: realsense_description/urdf/_d435.gazebo.xacro (robot description, xacro)
@@ -3,7 +3,4 @@
 <xacro:macro name="d435_realsense_gazebo"
   params="prefix color_width color_height color_update_rate depth_update_rate">
-  <gazebo reference="${prefix}camera_link">
-    <material value="Gazebo/Grey" />
-  </gazebo>
   <gazebo reference="${prefix}camera_color_frame">
     <sensor type="depth" name="${prefix}">

File: realsense_description/urdf/_d435.urdf.xacro (robot description, xacro)
@@ -39,5 +39,4 @@
           <mesh filename="package://realsense_description/meshes/visual/d435.dae" />
         </geometry>
-        <material name="grey"/>
       </visual>
       <collision>
